File: relay adapter board 16ch.kicad_pcb (KiCad board)
At the start: 2 copper layers, 13 parts, among them J1 RJ45_Shielded, J2 Screw_Terminal_01x02, J3 Conn_01x02_Pin, J4 Conn_02x10_Odd_Even, U3 TJA1051T-3

Commit message: Autosave
Parts:
- moved J4 19.9 mm to (112.0, 92.0), turned to 0 degrees
Changed lines of the file:
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@@
 	(footprint "Connector_PinSocket_2.54mm:PinSocket_2x10_P2.54mm_Vertical"
 		(layer "B.Cu")
-		(at 108.96 72.34 180)
+		(at 111.96 92)
 		(descr "Through hole straight socket strip, 2x10, 2.54mm pitch, double rows (from Kicad 4.0.7), script generated")
 		(tags "Through hole socket strip THT 2x10 2.54mm double row")
@@
 		(duplicate_pad_numbers_are_jumpers no)
 		(fp_line
+			(start -3.87 -24.19)
+			(end 1.33 -24.19)
+			(stroke
+				(width 0.12)
+				(type solid)
+			)
+			(layer "B.SilkS")
+		)
+		(fp_line
+			(start -3.87 1.33)
+			(end -3.87 -24.19)
+			(stroke
+				(width 0.12)
+				(type solid)
+			)
+			(layer "B.SilkS")
+		)
+		(fp_line
+			(start -3.87 1.33)
+			(end -1.27 1.33)
+			(stroke
+				(width 0.12)
+				(type solid)
+			)
+			(layer "B.SilkS")
+		)
+		(fp_line
+			(start -1.27 -1.27)
+			(end 1.33 -1.27)
+			(stroke
+				(width 0.12)
+				(type solid)
+			)
+			(layer "B.SilkS")
+		)
+		(fp_line
+			(start -1.27 1.33)
+			(end -1.27 -1.27)
+			(stroke
+				(width 0.12)
+				(type solid)
+			)
+			(layer "B.SilkS")
+		)
+		(fp_line
+			(start 0 1.33)
+			(end 1.33 1.33)
+			(stroke
+				(width 0.12)
+				(type solid)
+			)
+			(layer "B.SilkS")
+		)
+		(fp_line
+			(start 1.33 -1.27)
+			(end 1.33 -24.19)
+			(stroke
+				(width 0.12)
+				(type solid)
+			)
+			(layer "B.SilkS")
+		)
+		(fp_line
 			(start 1.33 1.33)
 			(end 1.33 0)
@@
 		)
 		(fp_line
-			(start 1.33 -1.27)
-			(end 1.33 -24.19)
-			(stroke
-				(width 0.12)
-				(type solid)
-			)
-			(layer "B.SilkS")
-		)
-		(fp_line
-			(start 0 1.33)
-			(end 1.33 1.33)
-			(stroke
-				(width 0.12)
-				(type solid)
-			)
-			(layer "B.SilkS")
-		)
-		(fp_line
-			(start -1.27 1.33)
-			(end -1.27 -1.27)
-			(stroke
-				(width 0.12)
-				(type solid)
-			)
-			(layer "B.SilkS")
-		)
-		(fp_line
-			(start -1.27 -1.27)
-			(end 1.33 -1.27)
-			(stroke
-				(width 0.12)
-				(type solid)
-			)
-			(layer "B.SilkS")
-		)
-		(fp_line
-			(start -3.87 1.33)
-			(end -1.27 1.33)
-			(stroke
-				(width 0.12)
-				(type solid)
-			)
-			(layer "B.SilkS")
-		)
-		(fp_line
-			(start -3.87 1.33)
-			(end -3.87 -24.19)
-			(stroke
-				(width 0.12)
-				(type solid)
-			)
-			(layer "B.SilkS")
-		)
-		(fp_line
-			(start -3.87 -24.19)
-			(end 1.33 -24.19)
-			(stroke
-				(width 0.12)
-				(type solid)
-			)
-			(layer "B.SilkS")
+			(start -4.31 -24.63)
+			(end -4.31 1.77)
+			(stroke
+				(width 0.05)
+				(type solid)
+			)
+			(layer "B.CrtYd")
+		)
+		(fp_line
+			(start -4.31 1.77)
+			(end 1.77 1.77)
+			(stroke
+				(width 0.05)
+				(type solid)
+			)
+			(layer "B.CrtYd")
+		)
+		(fp_line
+			(start 1.77 -24.63)
+			(end -4.31 -24.63)
+			(stroke
+				(width 0.05)
+				(type solid)
+			)
+			(layer "B.CrtYd")
 		)
 		(fp_line
@@
 		)
 		(fp_line
-			(start 1.77 -24.63)
-			(end -4.31 -24.63)
-			(stroke
-				(width 0.05)
-				(type solid)
-			)
-			(layer "B.CrtYd")
-		)
-		(fp_line
-			(start -4.31 1.77)
-			(end 1.77 1.77)
-			(stroke
-				(width 0.05)
-				(type solid)
-			)
-			(layer "B.CrtYd")
-		)
-		(fp_line
-			(start -4.31 -24.63)
-			(end -4.31 1.77)
-			(stroke
-				(width 0.05)
-				(type solid)
-			)
-			(layer "B.CrtYd")
+			(start -3.81 -24.13)
+			(end -3.81 1.27)
+			(stroke
+				(width 0.1)
+				(type solid)
+			)
+			(layer "B.Fab")
+		)
+		(fp_line
+			(start -3.81 1.27)
+			(end 0.27 1.27)
+			(stroke
+				(width 0.1)
+				(type solid)
+			)
+			(layer "B.Fab")
+		)
+		(fp_line
+			(start 0.27 1.27)
+			(end 1.27 0.27)
+			(stroke
+				(width 0.1)
+				(type solid)
+			)
+			(layer "B.Fab")
+		)
+		(fp_line
+			(start 1.27 -24.13)
+			(end -3.81 -24.13)
+			(stroke
+				(width 0.1)
+				(type solid)
+			)
+			(layer "B.Fab")
 		)
 		(fp_line
@@
 			(layer "B.Fab")
 		)
-		(fp_line
-			(start 1.27 -24.13)
-			(end -3.81 -24.13)
-			(stroke
-				(width 0.1)
-				(type solid)
-			)
-			(layer "B.Fab")
-		)
-		(fp_line
-			(start 0.27 1.27)
-			(end 1.27 0.27)
-			(stroke
-				(width 0.1)
-				(type solid)
-			)
-			(layer "B.Fab")
-		)
-		(fp_line
-			(start -3.81 1.27)
-			(end 0.27 1.27)
-			(stroke
-				(width 0.1)
-				(type solid)
-			)
-			(layer "B.Fab")
-		)
-		(fp_line
-			(start -3.81 -24.13)
-			(end -3.81 1.27)
-			(stroke
-				(width 0.1)
-				(type solid)
-			)
-			(layer "B.Fab")
-		)
 		(fp_text user "${REFERENCE}"
 			(at -1.27 -11.43 90)
@@
 		)
 		(pad "1" thru_hole rect
-			(at 0 0 180)
+			(at 0 0)
 			(size 1.7 1.7)
 			(drill 1)
@@
 		)
 		(pad "2" thru_hole circle
-			(at -2.54 0 180)
+			(at -2.54 0)
 			(size 1.7 1.7)
 			(drill 1)
@@
 		)
 		(pad "3" thru_hole circle
-			(at 0 -2.54 180)
+			(at 0 -2.54)
 			(size 1.7 1.7)
 			(drill 1)
@@
 		)
 		(pad "4" thru_hole circle
-			(at -2.54 -2.54 180)
+			(at -2.54 -2.54)
 			(size 1.7 1.7)
 			(drill 1)
@@
 		)
 		(pad "5" thru_hole circle
-			(at 0 -5.08 180)
+			(at 0 -5.08)
 			(size 1.7 1.7)
 			(drill 1)
@@
 		)
 		(pad "6" thru_hole circle
-			(at -2.54 -5.08 180)
+			(at -2.54 -5.08)
 			(size 1.7 1.7)
 			(drill 1)
@@
 		)
 		(pad "7" thru_hole circle
-			(at 0 -7.62 180)
+			(at 0 -7.62)
 			(size 1.7 1.7)
 			(drill 1)
@@
 		)
 		(pad "8" thru_hole circle
-			(at -2.54 -7.62 180)
+			(at -2.54 -7.62)
 			(size 1.7 1.7)
 			(drill 1)
@@
 		)
 		(pad "9" thru_hole circle
-			(at 0 -10.16 180)
+			(at 0 -10.16)
 			(size 1.7 1.7)
 			(drill 1)
@@
 		)
 		(pad "10" thru_hole circle
-			(at -2.54 -10.16 180)
+			(at -2.54 -10.16)
 			(size 1.7 1.7)
 			(drill 1)
@@
 		)
 		(pad "11" thru_hole circle
-			(at 0 -12.7 180)
+			(at 0 -12.7)
 			(size 1.7 1.7)
 			(drill 1)
@@
 		)
 		(pad "12" thru_hole circle
-			(at -2.54 -12.7 180)
+			(at -2.54 -12.7)
 			(size 1.7 1.7)
 			(drill 1)
@@
 		)
 		(pad "13" thru_hole circle
-			(at 0 -15.24 180)
+			(at 0 -15.24)
 			(size 1.7 1.7)
 			(drill 1)
@@
 		)
 		(pad "14" thru_hole circle
-			(at -2.54 -15.24 180)
+			(at -2.54 -15.24)
 			(size 1.7 1.7)
 			(drill 1)
@@
 		)
 		(pad "15" thru_hole circle
-			(at 0 -17.78 180)
+			(at 0 -17.78)
 			(size 1.7 1.7)
 			(drill 1)
@@
 		)
 		(pad "16" thru_hole circle
-			(at -2.54 -17.78 180)
+			(at -2.54 -17.78)
 			(size 1.7 1.7)
 			(drill 1)
@@
 		)
 		(pad "17" thru_hole circle
-			(at 0 -20.32 180)
+			(at 0 -20.32)
 			(size 1.7 1.7)
 			(drill 1)
@@
 		)
 		(pad "18" thru_hole circle
-			(at -2.54 -20.32 180)
+			(at -2.54 -20.32)
 			(size 1.7 1.7)
 			(drill 1)
@@
 		)
 		(pad "19" thru_hole circle
-			(at 0 -22.86 180)
+			(at 0 -22.86)
 			(size 1.7 1.7)
 			(drill 1)
@@
 		)
 		(pad "20" thru_hole circle
-			(at -2.54 -22.86 180)
-			(size 1.7 1.7)
-			(drill 1)
+			(at -2.54 -22.86)
+			(size 1.7 1.7)
+			(drill 1)
